Commit message: Added more complex 3d model. Specified some actual values in simulation_model

File: asv_pilot/data/emily.urdf (robot description, URDF)
Before this commit: robot emily, 1 links, 0 joints
Links:
- link base_link: geometry visual mesh filename=package://asv_pilot/data/emily2.dae

Commit message: Renamed the model

File: asv_pilot/data/emily.urdf (robot description, URDF)
Before this commit: robot emily, 1 links, 0 joints
Links:
- link base_link: geometry visual mesh filename=package://asv_pilot/data/emily.dae

Commit message: Added UWSim to launch

File: asv_pilot/data/emily.urdf (robot description, URDF)
Before this commit: robot emily, 1 links, 0 joints
Links:
- link base_link: geometry visual mesh filename=package://asv_pilot/data/emily.3ds
